File: Megavolt Rev2/Megavolt Rev2.kicad_pcb (KiCad board)
At the start: 2 copper layers, 105 x 50 mm, 87 parts, among them J1 DCIN, J2 GLIDE, J3 RESET, J4 ICSP, J5 CV, J6 GATE, J7 MIDI, Q1 MMBT5551L, Q2 MMBT5551L, U1 TL072, U2 MCP4822, U3 L78L10_SOT89, U4 ATMEGA328-AU, U5 TL074, U6 4504, U7 HCPL-0701, Y1 16MHz

Commit message: Rev.3 WIP
Parts:
- removed the C4 at (101.9, 104.6)
- removed H1, H2, H3, H4, H5, H6: MountingHole, MountingHole:MountingHole_3.2mm_M3_DIN965
- removed the R10 at (186.4, 99.0)
- removed the R11 at (186.4, 96.5)
- removed the R12 at (149.6, 85.6)
- removed the R13 at (152.1, 85.6)
- removed the R14 at (154.7, 85.6)
- removed the R15 at (157.2, 85.6)
- removed the R6 at (186.5, 109.2)
- removed the R7 at (186.4, 106.6)
- removed the R8 at (186.4, 104.1)
- removed the R9 at (186.4, 101.5)
- added C7: 1uF, Capacitor_SMD:C_0805_2012Metric, B.Cu at (-118.9, 83.1)
- added D1: 1N5819WS, Diode_SMD:D_SOD-323, B.Cu at (-104.6, 73.7)
- added D2: 1N5819WS, Diode_SMD:D_SOD-323, B.Cu at (-134.6, 77.4)
- added F1: 200mA@6V, Fuse:Fuse_0402_1005Metric, B.Cu at (-116.6, 81.9)
- added F2: 750mA@24V, Fuse:Fuse_1812_4532Metric, B.Cu at (-104.6, 77.2)
- added F3: 750mA@24V, Fuse:Fuse_1812_4532Metric, B.Cu at (-130.0, 77.2)
- added J10: AudioJack2, Dewdrop:Amphenol AJCM-MN-2, F.Cu at (-127.0, 139.7)
- added J11: AudioJack2, Dewdrop:Amphenol AJCM-MN-2, F.Cu at (-101.6, 139.7)
- added J12: AudioJack2, Dewdrop:Amphenol AJCM-MN-2, F.Cu at (-127.0, 165.1)
- added J13: AudioJack2, Dewdrop:Amphenol AJCM-MN-2, F.Cu at (-101.6, 165.1)
- added J8: AudioJack2, Dewdrop:Amphenol AJCM-MN-2, F.Cu at (-127.0, 114.3)
- added J9: AudioJack2, Dewdrop:Amphenol AJCM-MN-2, F.Cu at (-101.6, 114.3)
- added R25: 1k, Resistor_SMD:R_0603_1608Metric, B.Cu at (-103.3, 156.1)
- added R26: 1k, Resistor_SMD:R_0603_1608Metric, B.Cu at (-122.6, 154.5)
- added R27: 1k, Resistor_SMD:R_0603_1608Metric, B.Cu at (-133.3, 119.4)
- added R28: 1k, Resistor_SMD:R_0603_1608Metric, B.Cu at (-108.0, 118.9)
- added R29: 1k, Resistor_SMD:R_0603_1608Metric, B.Cu at (-133.5, 135.5)
- added R30: 1k, Resistor_SMD:R_0603_1608Metric, B.Cu at (-108.0, 144.5)
- added R31: 1k, Resistor_SMD:R_0603_1608Metric, B.Cu at (-113.0, 20.9)
- added R32: 1k, Resistor_SMD:R_0603_1608Metric, B.Cu at (-132.6, 66.0)
- added R33: 1k, Resistor_SMD:R_0603_1608Metric, B.Cu at (-108.0, 58.7)
- added RV3: R_Potentiometer_Small, Potentiometer_THT:Potentiometer_Alps_RK09L_Single_Vertical, F.Cu at (-129.5, 25.4)
- C1: renamed from C9; moved to B.Cu
- C10: renamed from C1; moved to B.Cu
- C11: renamed from C2; moved to B.Cu
- C12: renamed from C13; moved to B.Cu
- C13: renamed from C14; moved to B.Cu
- C14: renamed from C15; moved to B.Cu
- C15: renamed from C17; moved to B.Cu
- C16: renamed from C6; moved to B.Cu
- C17: renamed from C7; moved to B.Cu
- C18: renamed from C22; moved to B.Cu
- C19: renamed from C16; moved to B.Cu
- C2: renamed from C10; moved to B.Cu
- C20: renamed from C18; moved to B.Cu
- C21: renamed from C20; moved to B.Cu
- C22: renamed from C21; moved to B.Cu
- C23, C8, J1, J3, J4, Q1, Q2, U3, Y1: moved to B.Cu
- C3: renamed from C11; moved to B.Cu
- C4: renamed from C12; moved to B.Cu
- C5: renamed from C19; moved to B.Cu
- C6: renamed from C3; moved to B.Cu
- C9: renamed from C5; moved to B.Cu
- D3: renamed from D1; moved to B.Cu
- D4: renamed from D2; footprint Connector_PinHeader_2.54mm:PinHeader_1x02_P2.54mm_Vertical -> LED_THT:LED_D5.0mm
- D5: renamed from D3; footprint Connector_PinHeader_2.54mm:PinHeader_1x02_P2.54mm_Vertical -> LED_THT:LED_D5.0mm
- J2: value GLIDE -> DIN-5; footprint Connector_PinHeader_2.54mm:PinHeader_1x03_P2.54mm_Vertical -> Dewdrop:Switchcraft 57NC5FX
- J5: value CV -> AudioJack2; footprint Connector_PinHeader_2.54mm:PinHeader_1x07_P2.54mm_Vertical -> Dewdrop:Amphenol AJCM-MN-2
- J6: value GATE -> AudioJack2; footprint Connector_PinHeader_2.54mm:PinHeader_1x05_P2.54mm_Vertical -> Dewdrop:Amphenol AJCM-MN-2
- J7: value MIDI -> AudioJack2; footprint Connector_PinHeader_2.54mm:PinHeader_1x02_P2.54mm_Vertical -> Dewdrop:Amphenol AJCM-MN-2
- R1: renamed from R22; moved to B.Cu
- R10: renamed from R4; footprint Resistor_SMD:R_0402_1005Metric -> Resistor_SMD:R_0603_1608Metric; moved to B.Cu
- R11: renamed from R1; footprint Resistor_SMD:R_0402_1005Metric -> Resistor_SMD:R_0603_1608Metric; moved to B.Cu
- R12: renamed from R3; footprint Resistor_SMD:R_0402_1005Metric -> Resistor_SMD:R_0603_1608Metric; moved to B.Cu
- R13: renamed from R18; footprint Resistor_SMD:R_0402_1005Metric -> Resistor_SMD:R_0603_1608Metric; moved to B.Cu
- R14: renamed from R21; footprint Resistor_SMD:R_0402_1005Metric -> Resistor_SMD:R_0603_1608Metric; moved to B.Cu
- R15: renamed from R29; footprint Resistor_SMD:R_0402_1005Metric -> Resistor_SMD:R_0603_1608Metric; moved to B.Cu
- R16: renamed from R34; footprint Resistor_SMD:R_0402_1005Metric -> Resistor_SMD:R_0603_1608Metric; moved to B.Cu
- R17: renamed from R28; footprint Resistor_SMD:R_0402_1005Metric -> Resistor_SMD:R_0603_1608Metric; moved to B.Cu
- R18: renamed from R17; footprint Resistor_SMD:R_0402_1005Metric -> Resistor_SMD:R_0603_1608Metric; moved to B.Cu
- R19: renamed from R20; footprint Resistor_SMD:R_0402_1005Metric -> Resistor_SMD:R_0603_1608Metric; moved to B.Cu
- R2: renamed from R27; footprint Resistor_SMD:R_0402_1005Metric -> Resistor_SMD:R_0603_1608Metric; moved to B.Cu
- R20: renamed from R33; footprint Resistor_SMD:R_0402_1005Metric -> Resistor_SMD:R_0603_1608Metric; moved to B.Cu
- R21: renamed from R16; footprint Resistor_SMD:R_0402_1005Metric -> Resistor_SMD:R_0603_1608Metric; moved to B.Cu
- R22: renamed from R19; footprint Resistor_SMD:R_0402_1005Metric -> Resistor_SMD:R_0603_1608Metric; moved to B.Cu
- R23: renamed from R26; footprint Resistor_SMD:R_0402_1005Metric -> Resistor_SMD:R_0603_1608Metric; moved to B.Cu
- R24: renamed from R30; footprint Resistor_SMD:R_0402_1005Metric -> Resistor_SMD:R_0603_1608Metric; moved to B.Cu
- R3: renamed from R25; footprint Resistor_SMD:R_0402_1005Metric -> Resistor_SMD:R_0603_1608Metric; moved to B.Cu
- R4: renamed from R23; moved to B.Cu
- R5: renamed from R31; footprint Resistor_SMD:R_0805_2012Metric -> Resistor_SMD:R_0603_1608Metric; moved to B.Cu
- R6: renamed from R24; moved to B.Cu
- R7: renamed from R32; footprint Resistor_SMD:R_0805_2012Metric -> Resistor_SMD:R_0603_1608Metric; moved to B.Cu
- R8: renamed from R5; footprint Resistor_SMD:R_0402_1005Metric -> Resistor_SMD:R_0603_1608Metric; moved to B.Cu
- R9: renamed from R2; footprint Resistor_SMD:R_0402_1005Metric -> Resistor_SMD:R_0603_1608Metric; moved to B.Cu
- RV1, RV2: footprint Potentiometer_SMD:Potentiometer_Bourns_3314J_Vertical -> Potentiometer_SMD:Potentiometer_Bourns_3314G_Vertical; moved to B.Cu
- U1: renamed from U7; moved to B.Cu
- U2: renamed from U4; moved to B.Cu
- U4: renamed from U2; moved to B.Cu
- U5: renamed from U6; moved to B.Cu
- U6: renamed from U1; moved to B.Cu
- U7: renamed from U5; moved to B.Cu
- moved J5 302.2 mm to (-101.6, 20.3)
- moved R19 300.2 mm to (-126.1, 132.9), turned to -90 degrees
- moved R22 298.5 mm to (-124.3, 132.9), turned to -90 degrees
- moved C23 296.3 mm to (-125.1, 136.1), turned to 180 degrees
- moved R20 294.4 mm to (-126.1, 139.3), turned to 90 degrees
- moved C16 293.8 mm to (-118.7, 153.9)
- moved R24 292.8 mm to (-124.3, 139.3), turned to 90 degrees
- moved U7 291.1 mm to (-119.4, 136.1), turned to 180 degrees
- moved R21 289.5 mm to (-114.4, 132.9), turned to -90 degrees
- moved R18 287.9 mm to (-112.6, 132.9), turned to 90 degrees
- moved R3 286.9 mm to (-129.1, 183.8), turned to 0 degrees
- moved C9 285.6 mm to (-120.7, 34.9), turned to 180 degrees
- moved J6 284.9 mm to (-127.0, 62.2), turned to 0 degrees
- moved R23 283.9 mm to (-114.4, 139.3), turned to 90 degrees
- moved R17 282.3 mm to (-112.6, 139.3), turned to -90 degrees
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- renumbered LOGO2 to LOGO1, LOGO1 to LOGO2
Connections:
- D3 pad 2: Net-(D1-Pad2) -> Net-(D3-Pad2)
- J1 pad 1: +15V -> /+15V_raw
- J1 pad 3: +5V -> /+5V_raw
- J1 pad 5: -15V -> /-15V_raw
- J2 pad 1: +5V -> unconnected-(J2-Pad1)
- J2 pad 2: GLIDE_Out -> unconnected-(J2-Pad2)
- J2 pad 3: GND -> unconnected-(J2-Pad3)
- R3 pad 1: Net-(J7-Pad1) -> Net-(J2-Pad4)
- U1 pad 3: Net-(D1-Pad2) -> Net-(D3-Pad2)
- U2 pad 10: CV4_Sig -> CV3_Sig
- U2 pad 13: CV6_Sig -> CV4_Sig
- U2 pad 14: CV5_Sig -> CV6_Sig
- U2 pad 27: unconnected-(U4-Pad27) -> GATE5_Sig
- U2 pad 32: unconnected-(U4-Pad32) -> GATE6_Sig
- U2 pad 9: CV3_Sig -> CV5_Sig
- U5 pad 12: unconnected-(U6-Pad12) -> GATE5_Out
- U5 pad 15: unconnected-(U6-Pad15) -> GATE6_Out
- U5 pad 9: GATE4_Sig -> GND
Routing:
- net +5V: track 184.1 -> 280.6 mm, vias 7 -> 13
- net MIDI_RX: track 27.6 -> 109.4 mm, vias 0 -> 2
- net GLIDE_Out: track 10.4 -> 88.4 mm
- net DAC2_Out: track 5.67 -> 70.8 mm, vias 0 -> 2
- net CV2_Out: track 71.9 -> 7.50 mm
- net DAC1_Out: track 7.00 -> 68.8 mm, vias 0 -> 2
- net CV1_Out: track 68.6 -> 12.8 mm
- net +15V: track 181.6 -> 146.3 mm, vias 3 -> 4
- net GATE2_Out: track 2.16 -> 37.0 mm, vias 0 -> 2
- net GATE4_Sig: track 34.4 -> 0.00 mm
- net Net-(D5-Pad1): track 8.60 -> 42.7 mm, vias 0 -> 2
- net Net-(C21-Pad1): track 49.8 -> 15.9 mm
- net Net-(C20-Pad1): track 39.7 -> 7.56 mm
- net Net-(C19-Pad1): track 36.9 -> 7.49 mm
- net GATE3_Sig: track 39.0 -> 68.0 mm
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- added copper zone on B.Cu, net +5V
- added copper zone on F.Cu, net +5V
Other:
- board size 105 x 50 mm -> 48.5 x 203.2 mm
- board text added: "1/1'"
- board text added: "1/16'"
- board text added: "1V/OCT"
- board text added: "AUX"
- board text added: "BEND"
- board text added: "EXPR"
- board text added: "GATE"
- board text added: "GLIDE"
- board text added: "MIDI"
- board text added: "MODWHEEL"
- board text added: "VELOCITY"
- board text removed: "+15V"
- board text removed: "+5V"
- board text removed: "-15V"
- board text removed: "1"
- board text removed: "GND"
- board text removed: "NC"
- board text removed: "Rev. 2a"
