File: Megavolt Rev2/Megavolt Rev2.kicad_sch (KiCad schematic)
At the start: 87 parts, among them J1 DCIN, J2 GLIDE, J3 RESET, J4 ICSP, J5 CV, J6 GATE, J7 MIDI, Q1 MMBT5551L, Q2 MMBT5551L, U1 TL072, U2 MCP4822, U3 L78L10_SOT89, U4 ATMEGA328-AU, U5 TL074, U6 4504, U7 HCPL-0701, Y1 16MHz

Commit message: Rev.3 WIP
Parts:
- removed C4: 10uF, Capacitor_THT:CP_Radial_D5.0mm_P2.50mm, symbol Megavolt-Rev2-rescue:CP_Small-Device
- removed H1, H2, H3, H4, H5, H6: MountingHole, MountingHole:MountingHole_3.2mm_M3_DIN965, symbol Mechanical:MountingHole
- removed J2: GLIDE, Connector_PinHeader_2.54mm:PinHeader_1x03_P2.54mm_Vertical, symbol Connector_Generic:Conn_01x03
- removed J5: CV, Connector_PinHeader_2.54mm:PinHeader_1x07_P2.54mm_Vertical, symbol Connector_Generic:Conn_01x07
- removed J6: GATE, Connector_PinHeader_2.54mm:PinHeader_1x05_P2.54mm_Vertical, symbol Connector_Generic:Conn_01x05
- removed J7: MIDI, Connector_PinHeader_2.54mm:PinHeader_1x02_P2.54mm_Vertical, symbol Connector_Generic:Conn_01x02
- removed R10, R11, R12, R13, R14, R15, R6, R7, R8, R9: 1k, Resistor_SMD:R_0603_1608Metric, symbol Device:R
- added C7: 1uF, Capacitor_SMD:C_0805_2012Metric, symbol Device:C_Small
- added D1, D2: 1N5819WS, Diode_SMD:D_SOD-323, symbol Diode:1N5819WS
- added F1: 200mA@6V, Fuse:Fuse_0402_1005Metric, symbol Device:Polyfuse
- added F2, F3: 750mA@24V, Fuse:Fuse_1812_4532Metric, symbol Device:Polyfuse
- added J10, J11, J12, J13, J5, J6, J7, J8, J9: AudioJack2, Dewdrop:Amphenol AJCM-MN-2, symbol Connector:AudioJack2
- added J2: DIN-5, Dewdrop:Switchcraft 57NC5FX, symbol Connector:DIN-5
- added R25, R26, R27, R28, R29, R30, R31, R32, R33: 1k, Resistor_SMD:R_0603_1608Metric, symbol Device:R
- added RV3: R_Potentiometer_Small, Potentiometer_THT:Potentiometer_Alps_RK09L_Single_Vertical, symbol Device:R_Potentiometer_Small
- D4: renamed from D2; footprint Connector_PinHeader_2.54mm:PinHeader_1x02_P2.54mm_Vertical -> LED_THT:LED_D5.0mm
- D5: renamed from D3; footprint Connector_PinHeader_2.54mm:PinHeader_1x02_P2.54mm_Vertical -> LED_THT:LED_D5.0mm
- R10: renamed from R4; footprint Resistor_SMD:R_0402_1005Metric -> Resistor_SMD:R_0603_1608Metric
- R11: renamed from R1; footprint Resistor_SMD:R_0402_1005Metric -> Resistor_SMD:R_0603_1608Metric
- R12: renamed from R3; footprint Resistor_SMD:R_0402_1005Metric -> Resistor_SMD:R_0603_1608Metric
- R13: renamed from R18; footprint Resistor_SMD:R_0402_1005Metric -> Resistor_SMD:R_0603_1608Metric
- R14: renamed from R21; footprint Resistor_SMD:R_0402_1005Metric -> Resistor_SMD:R_0603_1608Metric
- R15: renamed from R29; footprint Resistor_SMD:R_0402_1005Metric -> Resistor_SMD:R_0603_1608Metric
- R16: renamed from R34; footprint Resistor_SMD:R_0402_1005Metric -> Resistor_SMD:R_0603_1608Metric
- R17: renamed from R28; footprint Resistor_SMD:R_0402_1005Metric -> Resistor_SMD:R_0603_1608Metric
- R18: renamed from R17; footprint Resistor_SMD:R_0402_1005Metric -> Resistor_SMD:R_0603_1608Metric
- R19: renamed from R20; footprint Resistor_SMD:R_0402_1005Metric -> Resistor_SMD:R_0603_1608Metric
- R2: renamed from R27; footprint Resistor_SMD:R_0402_1005Metric -> Resistor_SMD:R_0603_1608Metric
- R20: renamed from R33; footprint Resistor_SMD:R_0402_1005Metric -> Resistor_SMD:R_0603_1608Metric
- R21: renamed from R16; footprint Resistor_SMD:R_0402_1005Metric -> Resistor_SMD:R_0603_1608Metric
- R22: renamed from R19; footprint Resistor_SMD:R_0402_1005Metric -> Resistor_SMD:R_0603_1608Metric
- R23: renamed from R26; footprint Resistor_SMD:R_0402_1005Metric -> Resistor_SMD:R_0603_1608Metric
- R24: renamed from R30; footprint Resistor_SMD:R_0402_1005Metric -> Resistor_SMD:R_0603_1608Metric
- R3: renamed from R25; footprint Resistor_SMD:R_0402_1005Metric -> Resistor_SMD:R_0603_1608Metric
- R5: renamed from R31; footprint Resistor_SMD:R_0805_2012Metric -> Resistor_SMD:R_0603_1608Metric
- R7: renamed from R32; footprint Resistor_SMD:R_0805_2012Metric -> Resistor_SMD:R_0603_1608Metric
- R8: renamed from R5; footprint Resistor_SMD:R_0402_1005Metric -> Resistor_SMD:R_0603_1608Metric
- R9: renamed from R2; footprint Resistor_SMD:R_0402_1005Metric -> Resistor_SMD:R_0603_1608Metric
- RV1, RV2: footprint Potentiometer_SMD:Potentiometer_Bourns_3314J_Vertical -> Potentiometer_SMD:Potentiometer_Bourns_3314G_Vertical
- renumbered C9 to C1, C1 to C10, C2 to C11, C13 to C12, C14 to C13, C15 to C14, C17 to C15, C6 to C16, C7 to C17, C22 to C18, C16 to C19, C10 to C2, C18 to C20, C20 to C21, C21 to C22, C11 to C3, C12 to C4, C19 to C5, C3 to C6, C5 to C9, D1 to D3, LOGO2 to LOGO1, LOGO1 to LOGO2, R22 to R1, R23 to R4, R24 to R6, U7 to U1, U4 to U2, U2 to U4, U6 to U5, U1 to U6, U5 to U7
Connections:
- net +15V: now also D1.1 (K), F2.1; no longer J1.1 (Pin_1)
- net +5V: now also C7.1, F1.2, RV3.3; no longer J1.3 (Pin_3)
- net -15V: now also D2.2 (A), F3.2; no longer J1.5 (Pin_5)
- net CV1_Out: now also R25.1
- net CV2_Out: now also R26.1
- net CV3_Out: now also R27.1
- net CV3_Sig: now also U2.10 (PD6/PCINT22/OC0A/AIN0); no longer U2.9 (PD5/PCINT21/OC0B/T1)
- net CV4_Out: now also R28.1
- net CV4_Sig: now also U2.13 (PB1/PCINT1/OC1A); no longer U2.10 (PD6/PCINT22/OC0A/AIN0)
- net CV5_Out: now also R29.1
- net CV5_Sig: now also U2.9 (PD5/PCINT21/OC0B/T1); no longer U2.14 (PB2/PCINT2/~{SS}/OC1B)
- net CV6_Out: now also R30.1
- net CV6_Sig: now also U2.14 (PB2/PCINT2/~{SS}/OC1B); no longer U2.13 (PB1/PCINT1/OC1A)
- net GATE1_Out: now also R31.1
- net GATE2_Out: now also R32.1
- net GATE3_Out: now also R33.1
- net GATE4_Sig: no longer U5.9 (Din)
- net GLIDE_Out: now also RV3.2
- net GND: now also U5.9 (Din), C7.2, D1.2 (A), D2.1 (K), J10.S, J11.S, J12.S, J13.S, J5.S, J6.S, J7.S, J8.S, J9.S, RV3.1
- net at R3.1: now also J2.4
- net GATE5_Out: now reaches U5.12 (Eout)
- net GATE6_Out: now reaches U5.15 (Fout)
- net at D3.2 (A), U1.3 (C): now also J2.5
- net GATE5_Sig: now reaches U2.27 (PC4/ADC4/SDA/PCINT12)
- net GATE6_Sig: now reaches U2.32 (PD2/INT0/PCINT18)
- new net: J8.T, R27.2
- new net: J7.T, R33.2
- new net: J9.T, R28.2
- new net: J12.T, R25.2
- new net: J6.T, R32.2
- new net: J10.T, R29.2
- new net: J13.T, R26.2
- new net: J5.T, R31.2
- new net: J11.T, R30.2
- new net +15V_raw: F2.2, J1.1 (Pin_1)
- new net +5V_raw: F1.1, J1.3 (Pin_3)
- new net -15V_raw: F3.1, J1.5 (Pin_5)
- no-connect marks 0 -> 3
Other:
- moved on the sheet: C12, C13, C6, C8, C9, J1, J3, J4, R8, U3, Y1
