File: Megavolt_MIDI_CV.kicad_pcb (KiCad board)
At the start: 2 copper layers, 105 x 50 mm, 87 parts, among them J1 DCIN, J2 GLIDE, J3 RESET, J4 ICSP, J5 CV, J6 GATE, J7 MIDI, Q1 MMBT5551L, Q2 MMBT5551L, U1 TL072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

Commit message: Rev. 3 WIP
Parts:
- removed C15: 100nF, Capacitor_SMD:C_0603_1608Metric
- removed C4: 10uF, Capacitor_THT:CP_Radial_D5.0mm_P2.50mm
- removed C8: 22uF, Capacitor_THT:CP_Radial_D5.0mm_P2.50mm
- removed H3, H4: MountingHole_Pad, MountingHole:MountingHole_3.2mm_M3_DIN965_Pad
- removed J1: DCIN, Connector_Molex:Molex_KK-254_AE-6410-06A_1x06_P2.54mm_Vertical
- removed Q2: MMBT5551L, Package_TO_SOT_SMD:SOT-23
- added C24: 22uF, Capacitor_THT:CP_Radial_D6.3mm_P2.50mm, F.Cu at (101.6, 121.7)
- added C25: 22uF, Capacitor_THT:CP_Radial_D6.3mm_P2.50mm, F.Cu at (101.4, 91.4)
- added D20: 1N5817, Diode_SMD:D_SOD-123, F.Cu at (94.5, 112.8)
- added D21: 1N5817, Diode_SMD:D_SOD-123, F.Cu at (94.2, 90.3)
- added J11: Dotcom, Connector_Molex:Molex_KK-254_AE-6410-06A_1x06_P2.54mm_Vertical, F.Cu at (94.7, 107.7)
- added J8: Eurorack, Connector_PinHeader_2.54mm:PinHeader_2x08_P2.54mm_Vertical, F.Cu at (101.5, 97.6)
- added Q3: MMBT3904, Package_TO_SOT_SMD:SOT-23, F.Cu at (122.6, 90.0)
- added R35: 47k, Resistor_SMD:R_0402_1005Metric, F.Cu at (150.3, 98.2)
- added R36: 47k, Resistor_SMD:R_0402_1005Metric, F.Cu at (150.3, 99.4)
- C3: footprint Capacitor_THT:CP_Radial_D5.0mm_P2.50mm -> Capacitor_THT:CP_Radial_D6.3mm_P2.50mm
- J2: value GLIDE -> Glide
- J3: value RESET -> Reset
- J5: value CV -> CVs
- J6: value GATE -> GATEs
- Q1: value MMBT5551L -> MMBT3904
- U6: value 4504 -> LM324; footprint Package_SO:SOIC-16_3.9x9.9mm_P1.27mm -> Package_SO:SOIC-14_3.9x8.7mm_P1.27mm
- moved LOGO2 67.4 mm to (171.5, 119.3)
- moved U3 13.4 mm to (162.9, 91.6), turned to 180 degrees
- moved J2 13.4 mm to (139.6, 96.5)
- moved C16 9.86 mm to (149.1, 107.3)
- moved C18 9.86 mm to (149.1, 113.5)
- moved C20 9.86 mm to (149.1, 109.4)
- moved C21 9.86 mm to (149.1, 111.5)
- moved R18 9.86 mm to (146.3, 107.3)
- moved R21 9.86 mm to (146.3, 113.5)
- moved R29 9.86 mm to (146.4, 109.4)
- moved R34 9.86 mm to (146.3, 111.5)
- moved J4 8.69 mm to (129.2, 111.6)
- moved C3 8.08 mm to (108.8, 100.6), turned to 0 degrees
- moved C10 7.42 mm to (116.5, 101.4)
- moved C11 7.42 mm to (131.8, 104.4)
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Connections:
- net DAC1_SS renamed /DAC_SS
- net GLIDE_Out renamed /GLIDE
- net MIDI_RX renamed /MIDI_RX
- net RESET renamed /RESET
- net SPI_CLK renamed /SPI_CLK
- net SPI_MISO renamed /SPI_MISO
- net SPI_MOSI renamed /SPI_MOSI
- net XTAL1 renamed /XTAL1
- net XTAL2 renamed /XTAL2
- C3 pad 1: +15V -> +5V
- Q1 pad 3: Net-(D2-K) -> Net-(D3-K)
- R23 pad 1: Net-(Q1-B) -> Net-(Q3-B)
- R24 pad 1: Net-(Q2-B) -> Net-(Q1-B)
- U6 pad 1: +5V -> GATE1_Out
- U6 pad 10: GATE4_Out -> GATE3_Sig
- U6 pad 12: unconnected-(U6-Eout-Pad12) -> GATE4_Sig
- U6 pad 13: GND -> /2.5V_Ref
- U6 pad 14: GND -> GATE4_Out
- U6 pad 2: GATE1_Out -> /2.5V_Ref
- U6 pad 4: GATE2_Out -> +10V
- U6 pad 6: GATE3_Out -> /2.5V_Ref
- U6 pad 7: GATE3_Sig -> GATE2_Out
- U6 pad 8: GND -> GATE3_Out
- U6 pad 9: GATE4_Sig -> /2.5V_Ref
Routing:
- net +15V: track 179.3 -> 20.8 mm
- net -15V: track 96.1 -> 150.7 mm
- net /2.5V_Ref: track 0.00 -> 21.4 mm, vias 0 -> 5
- net Net-(D21-K): track 0.00 -> 17.5 mm
- net Net-(D20-A): track 0.00 -> 15.2 mm
- net CV1_Out: track 80.1 -> 67.5 mm
- net +5V: track 180.4 -> 193.0 mm, vias 7 -> 8
- net GATE1_Out: track 2.16 -> 13.4 mm, vias 0 -> 2
- net Net-(U5A-+): track 36.9 -> 27.1 mm
- net Net-(U5B-+): track 49.8 -> 40.0 mm
- net Net-(U5D-+): track 39.7 -> 29.8 mm
- net Net-(U5C-+): track 36.7 -> 26.9 mm
- net /MIDI_RX: track 27.6 -> 18.7 mm
- net GATE1_Sig: track 41.1 -> 32.8 mm
- net GND: track 16.5 -> 23.6 mm, vias 48 -> 15
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- added copper zone on In2.Cu, net +15V
- added copper zone on In1.Cu, net GND
Other:
- copper layers 2 -> 4
- board text added: "+"
- board text added: "-"
- board text added: "Interface"
- board text added: "MIDI-CV"
- board text added: "MidiVolt"
- board text added: "PWR"
- board text added: "Rev. 3"
- board text removed: "+15V"
- board text removed: "+5V"
- board text removed: "-15V"
- board text removed: "GND"
- board text removed: "MEGAVOLT MIDI-CV"
- board text removed: "NC"
- board text removed: "Rev. 2b"
