File: Megavolt_MIDI_CV.kicad_sch (KiCad schematic)
At the start: 87 parts, among them J1 DCIN, J2 GLIDE, J3 RESET, J4 ICSP, J5 CV, J6 GATE, J7 MIDI, Q1 MMBT5551L, Q2 MMBT5551L, U1 TL072, U2 MCP4822, U3 L78L10_SOT89, U4 ATMEGA328-AU, U5 TL074, U6 4504, U7 HCPL-0701, Y1 16MHz

Commit message: Rev. 3 WIP
Parts:
- removed C15: 100nF, Capacitor_SMD:C_0603_1608Metric, symbol Device:C_Small
- removed C3, C8: 22uF, Capacitor_THT:CP_Radial_D5.0mm_P2.50mm, symbol Megavolt-Rev2-rescue:CP_Small-Device
- removed C4: 10uF, Capacitor_THT:CP_Radial_D5.0mm_P2.50mm, symbol Megavolt-Rev2-rescue:CP_Small-Device
- removed H3, H4: MountingHole_Pad, MountingHole:MountingHole_3.2mm_M3_DIN965_Pad, symbol Mechanical:MountingHole_Pad
- removed J1: DCIN, Connector_Molex:Molex_KK-254_AE-6410-06A_1x06_P2.54mm_Vertical, symbol Connector_Generic:Conn_01x06
- removed Q1, Q2: MMBT5551L, Package_TO_SOT_SMD:SOT-23, symbol Transistor_BJT:MMBT5551L
- removed U6: 4504, Package_SO:SOIC-16_3.9x9.9mm_P1.27mm, symbol 4xxx:4504
- added C24, C25, C3: 22uF, Capacitor_THT:CP_Radial_D6.3mm_P2.50mm, symbol Device:C_Polarized_Small
- added D20, D21: 1N5817, Diode_SMD:D_SOD-123, symbol Diode:1N5817
- added J11: Dotcom, Connector_Molex:Molex_KK-254_AE-6410-06A_1x06_P2.54mm_Vertical, symbol Connector:Conn_01x06_Female
- added J8: Eurorack, Connector_PinHeader_2.54mm:PinHeader_2x08_P2.54mm_Vertical, symbol Connector:Conn_01x16_Pin
- added Q1, Q3: MMBT3904, Package_TO_SOT_SMD:SOT-23, symbol Transistor_BJT:MMBT3904
- added R35, R36: 47k, Resistor_SMD:R_0402_1005Metric, symbol Device:R_Small
- added U6: LM324, Package_SO:SOIC-14_3.9x8.7mm_P1.27mm, symbol Amplifier_Operational:LM324
- J2: value GLIDE -> Glide
- J3: value RESET -> Reset
- J5: value CV -> CVs
- J6: value GATE -> GATEs
Connections:
- net +10V: now also U6.4 (V+)
- net +15V: now also C24.1, D20.1 (K)
- net +5V: now also C3.1, J11.3 (Pin_3), J8.11 (Pin_11), J8.12 (Pin_12), R35.1
- net -15V: now also C25.2, D21.2 (A)
- net GATE1_Out: now also U6.1
- net GATE1_Sig: now also U6.3 (+)
- net GATE2_Out: now also U6.7
- net GATE2_Sig: now also U6.5 (+)
- net GATE3_Out: now also U6.8
- net GATE3_Sig: now also U6.10 (+)
- net GATE4_Out: now also U6.14
- net GATE4_Sig: now also U6.12 (+)
- net GND: now also C24.2, C25.1, C3.2, J11.4 (Pin_4), J8.3 (Pin_3), J8.4 (Pin_4), J8.5 (Pin_5), J8.6 (Pin_6), J8.7 (Pin_7), J8.8 (Pin_8), Q1.2 (E), Q3.2 (E), R36.1, U6.11 (V-)
- net at R23.1: now also Q3.1 (B)
- net at D2.1 (K): now also Q3.3 (C)
- net at R24.1: now also Q1.1 (B)
- net at D3.1 (K): now also Q1.3 (C)
- net DAC1_SS renamed DAC_SS
- net GLIDE_Out renamed GLIDE
- new net: D21.1 (K), J11.5 (Pin_5), J8.1 (Pin_1), J8.2 (Pin_2)
- new net: D20.2 (A), J11.1 (Pin_1), J8.10 (Pin_10), J8.9 (Pin_9)
- new net 2.5V_Ref: R35.2, R36.2, U6.13 (-), U6.2 (-), U6.6 (-), U6.9 (-)
- no-connect marks 6 -> 10
Other:
- note added: "Power Connector"
- note removed: "PSU"
- moved on the sheet: C17, C5, U3
